Commit message: add pochty final my_robot

File: task6/my_robot/robot_description/urdf/depth.urdf.xacro (robot description, xacro)
@@ -5,5 +5,5 @@
         <parent link="base_link"/>
         <child link="depth_frame"/>
-        <origin xyz="0.1 0 0.25" rpy="0 0 0"/>
+        <origin xyz="0.15 0.05 0.25" rpy="0 -0.3 0"/>
     </joint>
     <material name="aluminum">

File: task6/my_robot/robot_description/urdf/gazebo.urdf.xacro (robot description, xacro)
@@ -22,4 +22,13 @@
         </plugin>
         <plugin
+            filename="gz-sim-sensors-system"
+            name="gz::sim::systems::Sensors">
+        <render_engine>ogre2</render_engine>
+        </plugin>
+        <plugin
+            filename="gz-sim-imu-system"
+            name="gz::sim::systems::Imu">
+        </plugin>
+        <plugin
             filename="gz-sim-diff-drive-system"
             name="gz::sim::systems::DiffDrive">

Commit message: add probably final robot

File: task6/my_robot/robot_description/urdf/depth.urdf.xacro (robot description, xacro)
@@ -5,5 +5,5 @@
         <parent link="base_link"/>
         <child link="depth_frame"/>
-        <origin xyz="0.15 0.05 0.25" rpy="0 -0.3 0"/>
+        <origin xyz="0.15 0.05 0.25" rpy="0 0 0"/>
     </joint>
     <material name="aluminum">

File: task6/my_robot/robot_description/urdf/robot.urdf.xacro (robot description, xacro)
@@ -2,5 +2,5 @@
 <robot name='robot' xmlns:xacro="http://ros.org/wiki/xacro">
     <xacro:include filename="$(find robot_description)/urdf/gazebo.urdf.xacro" />
-    <xacro:include filename="$(find robot_description)/urdf/lidar.urdf.xacro" />
+    <!-- <xacro:include filename="$(find robot_description)/urdf/lidar.urdf.xacro" /> -->
     <xacro:include filename="$(find robot_description)/urdf/depth.urdf.xacro" />
     <xacro:include filename="$(find robot_description)/urdf/imu.urdf.xacro" />
